File: untitled.kicad_sch (KiCad schematic)
At the start: 66 parts, among them U1 K210_C913414, U12 PCIE-67P42H, U4 XC6206P182MR_C347373, U5 GD25LQ128EWIGR, U6 TMI7003C, U7 SGM803-TXN3/TR_C5152602, U8 XC6206P302MR_C347375, X1 X322526MMB4SI

Commit message: correcao de sch
Connections:
- net IO_4 is gone; now on net SPI_RX(42): U1.H11 (IO_4)
- net IO_5 is gone; now on net SPI_TX(40): U1.H12 (IO_5)
- net SPI_TX(40): now reaches U12.40
- net SPI_RX(42): now reaches U12.42
- net BOOT renamed BOOT(53)
- no-connect marks 44 -> 42
Changed lines of the file:
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@@
 	)
 	(no_connect
-		(at 325.12 137.16)
-	)
-	(no_connect
 		(at 325.12 119.38)
 	)
@@
 	)
 	(no_connect
-		(at 325.12 139.7)
-	)
-	(no_connect
 		(at 340.36 138.43)
 	)
@@
 	(wire
 		(pts
+			(xy 295.91 137.16) (xy 325.12 137.16)
+		)
+		(stroke
+			(width 0)
+			(type default)
+		)
+	)
+	(wire
+		(pts
 			(xy 147.32 127) (xy 142.24 127)
 		)
@@
 	(wire
 		(pts
+			(xy 295.91 139.7) (xy 325.12 139.7)
+		)
+		(stroke
+			(width 0)
+			(type default)
+		)
+	)
+	(wire
+		(pts
 			(xy 123.19 127) (xy 125.73 127)
 		)
@@
 		)
 	)
+	(label "IO_4"
+		(at 318.77 139.7 180)
+		(effects
+			(font
+				(size 1.27 1.27)
+			)
+			(justify right bottom)
+		)
+	)
 	(label "IO_18"
 		(at 96.52 83.82 0)
@@
 		)
 	)
+	(label "IO_5"
+		(at 318.77 137.16 180)
+		(effects
+			(font
+				(size 1.27 1.27)
+			)
+			(justify right bottom)
+		)
+	)
 	(label "F_D3"
 		(at 219.71 113.03 0)
@@
 		)
 	)
+	(label "UARTHS_RX"
+		(at 308.61 139.7 180)
+		(effects
+			(font
+				(size 1.27 1.27)
+			)
+			(justify right bottom)
+		)
+	)
 	(label "DVP_D5"
 		(at 163.83 48.26 0)
@@
 		)
 	)
+	(label "UARTHS_TX"
+		(at 308.61 137.16 180)
+		(effects
+			(font
+				(size 1.27 1.27)
+			)
+			(justify right bottom)
+		)
+	)
 	(label "F_D1"
 		(at 166.37 113.03 0)
@@
 		)
 	)
+	(hierarchical_label "SPI_TX(40)"
+		(shape bidirectional)
+		(at 295.91 137.16 180)
+		(effects
+			(font
+				(size 1.27 1.27)
+			)
+			(justify right)
+		)
+	)
+	(hierarchical_label "SPI_RX(42)"
+		(shape bidirectional)
+		(at 295.91 139.7 180)
+		(effects
+			(font
+				(size 1.27 1.27)
+			)
+			(justify right)
+		)
+	)
 	(hierarchical_label "PIN23"
 		(shape bidirectional)
@@
 		)
 	)
-	(hierarchical_label "BOOT"
+	(hierarchical_label "BOOT(53)"
 		(shape bidirectional)
 		(at 354.33 153.67 0)
